File: kicad/sm_2560_maket_board.sch (KiCad schematic (older format))
At the start: 13 parts

Commit message: Поправил макетное поле под новую версию платы SafeDuino 2560 ver 2.0.
Parts:
- added XP13: PLD-28, IWconnectors:PIN_ARRAY_14x2, symbol LFconnectors:connector_28pin_gost
- S1: value DTSGL-61K -> FSM1LP; footprint (none) -> IWsmd_case:SWD_BUTTON; symbol BUTTON_SMD_1 -> LFbutton:button_smd_1
- XP1, XP10, XP11, XP12, XP2, XP3, XP4, XP5, XP6, XP7, XP8, XP9: footprint ~ -> IWconnectors:PIN_ARRAY_8x1; symbol PIN_M_8 -> LFconnectors:connector_8pin_gost
Connections:
- net labels added: IOREF, MISO, MOSI, PC0, PC1, PC2, PC3, PC4, PC5, PC6, PC7, PD7, PG0, PG1, PG2, PL0, PL1, PL2, PL3, PL4, PL5, PL6, PL7, SCK, SS
- wire segments 99 -> 135
